Commit message: updated location of the meshes

File: kinematics_tests_support/urdf/kr210l150.urdf (robot description, URDF)
Before this commit: robot test_kuka_kr210, 8 links, 7 joints
Links:
- link Link1: geometry collision mesh filename=package://kinematics_tests_support/meshes/kr210l150/collisi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; visual mesh filename=package://kinematics_tests_support/meshes/kr210l150/visual/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
- link base_link: geometry collision mesh filename=package://kinematics_tests_support/meshes/kr210l150/collisi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; visual mesh filename=package://kinematics_tests_support/meshes/kr210l150/visual/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
- link link_2: geometry collision mesh filename=package://kinematics_tests_support/meshes/kr210l150/collisi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; visual mesh filename=package://kinematics_tests_support/meshes/kr210l150/visual/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
- link link_3: geometry collision mesh filename=package://kinematics_tests_support/meshes/kr210l150/collisi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; visual mesh filename=package://kinematics_tests_support/meshes/kr210l150/visual/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
- link link_4: geometry collision mesh filename=package://kinematics_tests_support/meshes/kr210l150/collisi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; visual mesh filename=package://kinematics_tests_support/meshes/kr210l150/visual/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
- link link_5: geometry collision mesh filename=package://kinematics_tests_support/meshes/kr210l150/collisi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; visual mesh filename=package://kinematics_tests_support/meshes/kr210l150/visual/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
- link link_6: geometry collision mesh filename=package://kinematics_tests_support/meshes/kr210l150/collisi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; visual mesh filename=package://kinematics_tests_support/meshes/kr210l150/visual/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

File: kinematics_tests_support/urdf/sia20d.urdf (robot description, URDF)
Before this commit: robot test_motoman_sia20d, 9 links, 8 joints
Links:
- link base_link: geometry collision mesh filename=package://kinematics_tests_support/meshes/sia20d/collision/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; visual mesh filename=package://kinematics_tests_support/meshes/sia20d/visual/MOT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
- link link_b: geometry collision mesh filename=package://kinematics_tests_support/meshes/sia20d/collision/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; visual mesh filename=package://kinematics_tests_support/meshes/sia20d/visual/MOT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
- link link_e: geometry collision mesh filename=package://kinematics_tests_support/meshes/sia20d/collision/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; visual mesh filename=package://kinematics_tests_support/meshes/sia20d/visual/MOT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
- link link_l: geometry collision mesh filename=package://kinematics_tests_support/meshes/sia20d/collision/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; visual mesh filename=package://kinematics_tests_support/meshes/sia20d/visual/MOT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
- link link_r: geometry collision mesh filename=package://kinematics_tests_support/meshes/sia20d/collision/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; visual mesh filename=package://kinematics_tests_support/meshes/sia20d/visual/MOT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
- link link_s: geometry collision mesh filename=package://kinematics_tests_support/meshes/sia20d/collision/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; visual mesh filename=package://kinematics_tests_support/meshes/sia20d/visual/MOT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
- link link_t: geometry collision mesh filename=package://kinematics_tests_support/meshes/sia20d/collision/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; visual mesh filename=package://kinematics_tests_support/meshes/sia20d/visual/MOT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
- link link_u: geometry collision mesh filename=package://kinematics_tests_support/meshes/sia20d/collision/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; visual mesh filename=package://kinematics_tests_support/meshes/sia20d/visual/MOT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
